File: effecitveRangeMic.kicad_pcb (KiCad board)
At the start: 2 copper layers, 24.4 x 18 mm, 27 parts, among them J1 MicHeader

Commit message: fix: drc check for font size
Other:
- board text added: "www.effective-range.com"
- board text removed: "www.effective-range.com/ products/micdevice"
Changed lines of the file:
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@@
 		)
 	)
-	(gr_text "www.effective-range.com/\nproducts/micdevice"
+	(gr_text "www.effective-range.com"
 		(at 119.137128 67.1322 0)
 		(layer "F.SilkS" knockout)
 		(effects
 			(font
-				(size 0.35 0.35)
-				(thickness 0.0875)
-				(bold yes)
+				(size 0.4 0.4)
+				(thickness 0.1)
 			)
 			(justify left bottom)

Commit message: Bumping release from 2.2.0 to 2.2.1
Other:
- board text added: "MicDevice v2.2.1"
- board text removed: "MicDevice v2.2.0"
Changed lines of the file:
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@@
 	(title_block
 		(title "Effective Range  Mic")
-		(date "2024-04-16")
-		(rev "2.2.0")
+		(date "2024-06-16")
+		(rev "2.2.1")
 		(company "Global Scope Ltd")
 		(comment 1 "Author: Ferenc Janky")
@@
 		(layer "Edge.Cuts")
 	)
-	(gr_text "MicDevice v2.2.0"
+	(gr_text "MicDevice v2.2.1"
 		(at 119.9896 60.9346 90)
 		(layer "B.Cu")
