File: effecitveRangeMic.kicad_pcb (KiCad board)
At the start: 2 copper layers, 24.4 x 18 mm, 27 parts, among them J1 MicHeader

Commit message: Bumping release from 2.2.1 to 2.2.2
Other:
- board text added: "MicDevice v2.2.2"
- board text removed: "MicDevice v2.2.1"
Changed lines of the file:
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@@
 		(title "Effective Range  Mic")
 		(date "2024-06-16")
-		(rev "2.2.1")
+		(rev "2.2.2")
 		(company "Global Scope Ltd")
 		(comment 1 "Author: Ferenc Janky")
@@
 		(layer "Edge.Cuts")
 	)
-	(gr_text "MicDevice v2.2.1"
+	(gr_text "MicDevice v2.2.2"
 		(at 119.9896 60.9346 90)
 		(layer "B.Cu")

Commit message: fix: qr url, stencil
Parts:
- removed the G*** at (140.8, 65.0)
- removed the G*** at (123.5, 66.5)

Commit message: Bumping release from 2.2.2 to 2.3.0
Other:
- board text added: "MicDevice v2.3.0"
- board text removed: "MicDevice v2.2.2"
Changed lines of the file:
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@@
 	(title_block
 		(title "Effective Range  Mic")
-		(date "2024-06-16")
-		(rev "2.2.2")
+		(date "2024-07-24")
+		(rev "2.3.0")
 		(company "Global Scope Ltd")
 		(comment 1 "Author: Ferenc Janky")
@@
 		(layer "Edge.Cuts")
 	)
-	(gr_text "MicDevice v2.2.2"
+	(gr_text "MicDevice v2.3.0"
 		(at 119.9896 60.9346 90)
 		(layer "B.Cu")
