File: effecitveRangeMic.kicad_sch (KiCad schematic)
At the start: 22 parts, among them J1 MicHeader

Commit message: updated kicad file version
Changed lines of the file:
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@@
 (kicad_sch
-	(version 20231120)
+	(version 20250114)
 	(generator "eeschema")
-	(generator_version "8.0")
+	(generator_version "9.0")
 	(paper "A4")
 	(title_block
@@
 		(comment 4 "Design Engineer: Ferenc Janky")
 	)
+	(rectangle
+		(start 195.58 82.55)
+		(end 217.17 104.14)
+		(stroke
+			(width 0.2)
+			(type dash)
+		)
+		(fill
+			(type none)
+		)
+	)
+	(text "BOM-only"
+		(exclude_from_sim no)
+		(at 210.312 85.09 0)
+		(effects
+			(font
+				(size 1.27 1.27)
+			)
+		)
+	)
 	(junction
 		(at 185.42 72.39)
@@
 		)
 	)
-	(rectangle
-		(start 195.58 82.55)
-		(end 217.17 104.14)
-		(stroke
-			(width 0.2)
-			(type dash)
-		)
-		(fill
-			(type none)
-		)
-	)
-	(text "BOM-only"
-		(exclude_from_sim no)
-		(at 210.312 85.09 0)
+	(label "SEL"
+		(at 139.7 85.09 0)
 		(effects
 			(font
 				(size 1.27 1.27)
 			)
-		)
-	)
-	(label "SEL"
-		(at 139.7 85.09 0)
-		(fields_autoplaced yes)
+			(justify left bottom)
+		)
+	)
+	(label "I2S_DIN"
+		(at 77.47 73.66 0)
 		(effects
 			(font
@@
 		)
 	)
-	(label "I2S_DIN"
-		(at 77.47 73.66 0)
-		(fields_autoplaced yes)
+	(label "I2S_FS"
+		(at 77.47 68.58 0)
 		(effects
 			(font
@@
 		)
 	)
-	(label "I2S_FS"
-		(at 77.47 68.58 0)
-		(fields_autoplaced yes)
+	(label "I2S_CLK"
+		(at 77.47 71.12 0)
 		(effects
 			(font
@@
 		)
 	)
-	(label "I2S_CLK"
-		(at 77.47 71.12 0)
-		(fields_autoplaced yes)
-		(effects
-			(font
-				(size 1.27 1.27)
-			)
-			(justify left bottom)
-		)
-	)
 	(label "DATA"
 		(at 116.84 73.66 180)
-		(fields_autoplaced yes)
 		(effects
 			(font
@@
 		)
 	)
+	(embedded_fonts no)
 )
